Commit message: add moveit_config

File: sitl_config/urdf/iris_arm_base.xacro (robot description, xacro)
@@ -177,10 +177,9 @@
     </xacro:bag_plugin_macro>
   </xacro:if>
-  <xacro:robotic_arm/>
   <!--Arm connect joint-->
   <joint name="arm_connect_joint" type="fixed">
-    <origin xyz="" rpy=""/>
+    <origin xyz="0 0 -0.05" rpy="0 ${M_PI} 0"/>
     <parent link="base_link"/>
-    <child link="toe"/>
+    <child link="link0"/>
   </joint>
 </robot>

File: sitl_config/urdf/robotic_arm.xacro (robot description, xacro)
@@ -1,122 +1,344 @@
 <?xml version="1.0"?>
-<robot xmlns:xacro="http://www.ros.org/wiki/xacro">
-<xacro:macro name="robotic_arm">
-  <xacro:property name="PI" value="3.14159265359"/>
-  <!-- Joints Control in Gazebo -->
-  <gazebo>
-    <plugin name="gazebo_ros_control" filename="libgazebo_ros_control.so"/>
-  </gazebo>
-  <!-- Geometrical properties -->
-  <xacro:property name="link_side" value="0.02"/>
-  <xacro:property name="joint_radius" value="0.018"/>
-  <xacro:property name="joint_length" value="0.025"/>
-  <xacro:property name="toe_length" value="0.03"/>
-  <xacro:property name="foot_length" value="0.04"/>
-  <xacro:property name="leg_length" value="0.10"/>
-  <xacro:property name="arm_length" value="0.10"/>
-  <xacro:property name="hand_length" value="0.04"/>
-  <xacro:property name="finger_length" value="0.03"/>
-  <!-- Materials -->
-  <material name="orange">
-    <color rgba="1.00 0.67 0.02 1.00"/>
-  </material>
-  <material name="gray">
-    <color rgba="0.80 0.80 0.80 1.00"/>
-  </material>
-  <!-- Generates a box visual/collision/inertial -->
-  <xacro:macro name="prism_vci" params="side length mass:=0.01 *origin">
-    <xacro:macro name="prism_geometry">
-      <xacro:insert_block name="origin"/>
-      <geometry>
-        <box size="${side} ${side} ${length}"/>
-      </geometry>
+<robot name="arm" xmlns:xacro="http://ros.org/wiki/xacro">
+    <!-- Defining the colors used in this robot -->
+    <material name="Black">
+        <color rgba="0 0 0 1"/>
+    </material>
+    <material name="White">
+        <color rgba="1 1 1 1"/>
+    </material>
+    <material name="Blue">
+        <color rgba="0 0 1 1"/>
+    </material>
+    <material name="Red">
+        <color rgba="1 0 0 1"/>
+    </material>
+    <!-- Constants -->
+    <xacro:property name="M_PI" value="3.14159"/>
+    <!-- link1 properties -->
+    <xacro:property name="link1_width" value="0.03" />
+    <xacro:property name="link1_len" value="0.10" />
+    <!-- link2 properties -->
+    <xacro:property name="link2_width" value="0.03" />
+    <xacro:property name="link2_len" value="0.14" />
+    <!-- link3 properties -->
+    <xacro:property name="link3_width" value="0.03" />
+    <xacro:property name="link3_len" value="0.22" />
+    <!-- link4 properties -->
+    <xacro:property name="link4_width" value="0.025" />
+    <xacro:property name="link4_len" value="0.06" />
+    <!-- link5 properties -->
+    <xacro:property name="link5_width" value="0.03" />
+    <xacro:property name="link5_len" value="0.06" />
+    <!-- link6 properties -->
+    <xacro:property name="link6_width" value="0.04" />
+    <xacro:property name="link6_len" value="0.02" />
+    <!-- Left gripper -->
+    <xacro:property name="left_gripper_len" value="0.08" />
+    <xacro:property name="left_gripper_width" value="0.01" />
+    <xacro:property name="left_gripper_height" value="0.01" />
+    <!-- Right gripper -->
+    <xacro:property name="right_gripper_len" value="0.08" />
+    <xacro:property name="right_gripper_width" value="0.01" />
+    <xacro:property name="right_gripper_height" value="0.01" />
+    <!-- Gripper frame -->
+    <xacro:property name="grasp_frame_radius" value="0.001" />
+    <!-- Inertial matrix -->
+    <xacro:macro name="inertial_matrix" params="mass">
+        <inertial>
+            <mass value="${mass}" />
+            <inertia ixx="1.0" ixy="0.0" ixz="0.0" iyy="0.5" iyz="0.0" izz="1.0" />
+        </inertial>
     </xacro:macro>
-    <visual>
-      <xacro:prism_geometry/>
-      <material name="orange"/>
-    </visual>
-    <collision>
-      <xacro:prism_geometry/>
-    </collision>
-    <inertial>
-      <xacro:insert_block name="origin"/>
-      <mass value="${mass}"/>
-      <inertia ixx="${(mass/12)*(side*side+length*length)}"
-               iyy="${(mass/12)*(side*side+length*length)}"
-               izz="${(mass/6)*(side*side)}"
-               ixy="0" ixz="0" iyz="0"/>
-    </inertial>
-  </xacro:macro>
-  <!-- Generates a cylinder visual/collision -->
-  <xacro:macro name="cylinder_vc" params="radius length *origin">
-    <xacro:macro name="cylinder_geometry">
-      <xacro:insert_block name="origin"/>
-      <geometry>
-        <cylinder length="${length}" radius="${radius}"/>
-      </geometry>
+    <!-- ///////////////////////////////////////   bottom_joint   //////////////////////////////////////////
+    <joint name="bottom_joint" type="fixed">
+        <origin xyz="0 0 0" rpy="0 0 0" />
+        <parent link="link0"/>
+        <child link="bottom_link"/>
+    </joint>
+    <link name="bottom_link">
+        <visual>
+              <origin xyz=" 0 0 -0.02"  rpy="0 0 0"/>
+                  <geometry>
+                       <box size="1 1 0.02" />
+                  </geometry>
+              <material name="Brown" />
+        </visual>
+        <collision>
+            <origin xyz=" 0 0 -0.02"  rpy="0 0 0"/>
+            <geometry>
+                <box size="1 1 0.02" />
+            </geometry>
+        </collision>
+        <xacro:inertial_matrix mass="500"/>
+    </link>
+-->
+    <!-- /////////////////////////////////////   BASE LINK    ////////////////////////////////////////////// -->
+    <link name="link0">
+        <visual>
+            <origin xyz="0 0 0" rpy="0 0 0" />
+            <geometry>
+                <box size="0.1 0.1 0.04" />
+            </geometry>
+            <material name="White" />
+        </visual>
+        <collision>
+            <origin xyz="0 0 0" rpy="0 0 0" />
+            <geometry>
+                <box size="0.1 0.1 0.04" />
+            </geometry>
+        </collision>
+        <xacro:inertial_matrix mass="1"/>
+    </link>
+    <joint name="joint1" type="revolute">
+        <parent link="link0"/>
+        <child link="link1"/>
+        <origin xyz="0 0 0.02" rpy="0 ${M_PI/2} 0" />
+        <axis xyz="-1 0 0" />
+        <limit effort="300" velocity="1" lower="-2.96" upper="2.96"/>
+        <dynamics damping="50" friction="1"/>
+    </joint>
+    <!-- /////////////////////////////////////   LINK1  ////////////////////////////////////////////// -->
+    <link name="link1" >
+        <visual>
+            <origin xyz="-${link1_len/2} 0 0" rpy="0 ${M_PI/2} 0" />
+            <geometry>
+                <cylinder radius="${link1_width}" length="${link1_len}"/>
+            </geometry>
+            <material name="Blue" />
+        </visual>
+        <collision>
+            <origin xyz="-${link1_len/2} 0 0" rpy="0 ${M_PI/2} 0" />
+            <geometry>
+                <cylinder radius="${link1_width}" length="${link1_len}"/>
+            </geometry>
+        </collision>
+        <xacro:inertial_matrix mass="1"/>
+    </link>
+    <joint name="joint2" type="revolute">
+        <parent link="link1"/>
+        <child link="link2"/>
+        <origin xyz="-${link1_len} 0 0.0" rpy="-${M_PI/2} 0 ${M_PI/2}" />
+        <axis xyz="1 0 0" />
+        <limit effort="300" velocity="1" lower="-2.35" upper="2.35" />
+        <dynamics damping="50" friction="1"/>
+    </joint>
+    <!-- ///////////////////////////////////////   LINK2  ////////////////////////////////////////////// -->
+    <link name="link2" >
+        <visual>
+            <origin xyz="0 0 ${link2_len/2}" rpy="0 0 0" />
+            <geometry>
+                <cylinder radius="${link2_width}" length="${link2_len}"/>
+            </geometry>
+            <material name="White" />
+        </visual>
+        <collision>
+            <origin xyz="0 0 ${link2_len/2}" rpy="0 0 0" />
+            <geometry>
+                <cylinder radius="${link2_width}" length="${link2_len}"/>
+            </geometry>
+        </collision>
+        <xacro:inertial_matrix mass="1"/>
+    </link>
+    <joint name="joint3" type="revolute">
+        <parent link="link2"/>
+        <child link="link3"/>
+        <origin xyz="0 0 ${link2_len}" rpy="0 ${M_PI} 0" />
+        <axis xyz="-1 0 0" />
+        <limit effort="300" velocity="1" lower="-2.62" upper="2.62" />
+        <dynamics damping="50" friction="1"/>
+    </joint>
+    <!-- /////////////////////////////////   LINK3  ///////////////////////////////////////////////////// -->
+    <link name="link3" >
+        <visual>
+            <origin xyz="0 0 -${link3_len/2}" rpy="0 0 0" />
+            <geometry>
+                <cylinder radius="${link3_width}" length="${link3_len}"/>
+            </geometry>
+            <material name="Blue" />
+        </visual>
+        <collision>
+            <origin xyz="0 0 -${link3_len/2}" rpy="0 0 0" />
+            <geometry>
+                <cylinder radius="${link3_width}" length="${link3_len}"/>
+            </geometry>
+        </collision>
+        <xacro:inertial_matrix mass="1"/>
+    </link>
+    <joint name="joint4" type="revolute">
+        <parent link="link3"/>
+        <child link="link4"/>
+        <origin xyz="0.0 0.0 -${link3_len}" rpy="0 ${M_PI/2} ${M_PI}" />
+        <axis xyz="1 0 0" />
+        <limit effort="300" velocity="1" lower="-2.62" upper="2.62" />
+        <dynamics damping="50" friction="1"/>
+    </joint>
+    <!-- ///////////////////////////////////   LINK4  //////////////////////////////////////////////// -->
+    <link name="link4" >
+        <visual>
+            <origin xyz="${link4_len/2} 0 0" rpy="0 ${M_PI/2} 0" />
+            <geometry>
+                <cylinder radius="${link4_width}" length="${link4_len}"/>
+            </geometry>
+            <material name="Black" />
+        </visual>
+        <collision>
+            <origin xyz="${link4_len/2} 0 0" rpy="0 ${M_PI/2} 0" />
+            <geometry>
+                <cylinder radius="${link4_width}" length="${link4_len}"/>
+            </geometry>
+        </collision>
+        <xacro:inertial_matrix mass="1"/>
+    </link>
+    <joint name="joint5" type="revolute">
+        <parent link="link4"/>
+        <child link="link5"/>
+        <origin xyz="${link4_len} 0.0 0.0" rpy="0 ${M_PI/2} 0" />
+        <axis xyz="1 0 0" />
+        <limit effort="300" velocity="1" lower="-2.62" upper="2.62" />
+        <dynamics damping="50" friction="1"/>
+    </joint>
+    <!-- //////////////////////////////////   LINK5  ///////////////////////////////////////////////// -->
+    <link name="link5">
+        <visual>
+            <origin xyz="0 0 ${link4_len/2}" rpy="0 0 0" />
+            <geometry>
+                <cylinder radius="${link5_width}" length="${link5_len}"/>
+            </geometry>
+            <material name="White" />
+        </visual>
+        <collision>
+            <origin xyz="0 0 ${link4_len/2} " rpy="0 0 0" />
+            <geometry>
+                <cylinder radius="${link5_width}" length="${link5_len}"/>
+            </geometry>
+        </collision>
+        <xacro:inertial_matrix mass="1"/>
+    </link>
+    <joint name="joint6" type="revolute">
+        <parent link="link5"/>
+        <child link="link6"/>
+        <origin xyz="0 0 ${link4_len}" rpy="${1.5*M_PI} -${M_PI/2} 0" />
+        <axis xyz="1 0 0" />
+        <limit effort="300" velocity="1" lower="-6.28" upper="6.28" />
+        <dynamics damping="50" friction="1"/>
+    </joint>
+    <!-- ////////////////////////////////   LINK6  ///////////////////////////////////////////////// -->
+    <link name="link6">
+        <visual>
+            <origin xyz="${link6_len/2} 0 0 " rpy="0 ${M_PI/2} 0" />
+            <geometry>
+                <cylinder radius="${link6_width}" length="${link6_len}"/>
+            </geometry>
+            <material name="Blue" />
+        </visual>
+        <collision>
+            <origin xyz="${link6_len/2} 0 0" rpy="0 ${M_PI/2} 0" />
+            <geometry>
+                <cylinder radius="${link6_width}" length="${link6_len}"/>
+            </geometry>
+        </collision>
+        <xacro:inertial_matrix mass="1"/>
+    </link>
+    <joint name="finger_joint1" type="prismatic">
+        <parent link="link6"/>
+        <child link="gripper_finger_link1"/>
+        <origin xyz="0.0 0 0" />
+        <axis xyz="0 1 0" />
+        <limit effort="100" lower="0" upper="0.06" velocity="1.0"/>
+        <dynamics damping="50" friction="1"/>
+    </joint>
+    <!-- //////////////////////////////////////   gripper   ////////////////////////////////////////////// -->
+    <!-- LEFT GRIPPER AFT LINK -->
+    <link name="gripper_finger_link1">
+        <visual>
+            <origin xyz="0.04 -0.03 0"/>
+            <geometry>
+                <box size="${left_gripper_len} ${left_gripper_width} ${left_gripper_height}" />
+            </geometry>
+            <material name="White" />
+        </visual>
+        <xacro:inertial_matrix mass="1"/>
+    </link>
+    <joint name="finger_joint2" type="fixed">
+        <parent link="link6"/>
+        <child link="gripper_finger_link2"/>
+        <origin xyz="0.0 0 0" />
+    </joint>
+    <!-- RIGHT GRIPPER AFT LINK -->
+    <link name="gripper_finger_link2">
+        <visual>
+            <origin xyz="0.04 0.03 0"/>
+            <geometry>
+                <box size="${right_gripper_len} ${right_gripper_width} ${right_gripper_height}" />
+            </geometry>
+            <material name="White" />
+        </visual>
+        <xacro:inertial_matrix mass="1"/>
+    </link>
+    <!-- Grasping frame -->
+    <link name="grasping_frame"/>
+    <joint name="grasping_frame_joint" type="fixed">
+      <parent link="link6"/>
+      <child link="grasping_frame"/>
+      <origin xyz="0.08 0 0" rpy="0 0 0"/>
+    </joint>
+    <!-- /////////////////////////////////   Gazebo   //////////////////////////////////////
+    <gazebo reference="bottom_link">
+        <material>Gazebo/White</material>
+    </gazebo>
+    -->
+    <gazebo reference="link0">
+        <material>Gazebo/White</material>
+    </gazebo>
+    <gazebo reference="link1">
+        <material>Gazebo/Blue</material>
+    </gazebo>
+    <gazebo reference="link2">
+        <material>Gazebo/White</material>
+    </gazebo>
+    <gazebo reference="link3">
+        <material>Gazebo/Blue</material>
+    </gazebo>
+    <gazebo reference="link4">
+        <material>Gazebo/Black</material>
+    </gazebo>
+    <gazebo reference="link5">
+        <material>Gazebo/White</material>
+    </gazebo>
+    <gazebo reference="link6">
+        <material>Gazebo/Blue</material>
+    </gazebo>
+    <gazebo reference="gripper_finger_link1">
+        <material>Gazebo/White</material>
+    </gazebo>
+    <gazebo reference="gripper_finger_link2">
+        <material>Gazebo/White</material>
+    </gazebo>
+    <!-- Transmissions for ROS Control -->
+    <xacro:macro name="transmission_block" params="joint_name">
+        <transmission name="tran1">
+            <type>transmission_interface/SimpleTransmission</type>
+            <joint name="${joint_name}">
+                <hardwareInterface>hardware_interface/PositionJointInterface</hardwareInterface>
+            </joint>
+            <actuator name="motor1">
+                <hardwareInterface>hardware_interface/PositionJointInterface</hardwareInterface>
+                <mechanicalReduction>1</mechanicalReduction>
+            </actuator>
+        </transmission>
     </xacro:macro>
-    <visual>
-      <xacro:cylinder_geometry/>
-      <material name="gray"/>
-    </visual>
-    <collision>
-      <xacro:cylinder_geometry/>
-    </collision>
-  </xacro:macro>
-  <!-- Generates child joint of parent -->
-  <xacro:macro name="arm_joint" params="child parent dist:=0 axis">
-    <joint name="${parent}_${child}_joint" type="revolute">
-      <origin xyz="0 0 ${dist}" rpy="0 0 0"/>
-      <parent link="${parent}"/>
-      <child link="${child}"/>
-      <axis xyz="${axis}"/>
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